File: circuit/msgeq7-simple.brd (EAGLE design)
At the start: 100 x 80 mm, 30 parts, among them IC1 LM3915N, IC2 MSGEQ7, Q1 BS250, Q2 BS250, Q3 BS250, Q4 BS250, Q5 BS250, Q6 BS250, Q7 BS250, X1 KLBR4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

Commit message: fixed location of R12
Connections:
- net GND: no longer R12.P$2
- net N$15: now also R12.P$2
Changed lines of the file:
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@@
 <contactref element="X1" pad="S"/>
 <contactref element="C3" pad="1"/>
-<contactref element="R12" pad="P$2"/>
 <contactref element="C4" pad="1"/>
 <contactref element="R14" pad="P$2"/>
@@
 <contactref element="U$1" pad="10"/>
 <contactref element="X2" pad="S"/>
-<wire x1="5.08" y1="24.13" x2="66.04" y2="16.51" width="0" layer="19" extent="1-1"/>
-<wire x1="90.17" y1="35.56" x2="5.08" y2="24.13" width="0" layer="19" extent="1-1"/>
-<wire x1="27.94" y1="16.51" x2="90.17" y2="35.56" width="0" layer="19" extent="1-1"/>
+<wire x1="88.59" y1="28.87" x2="90.17" y2="35.56" width="0" layer="19" extent="1-1"/>
+<wire x1="88.59" y1="12.36" x2="88.59" y2="28.87" width="0" layer="19" extent="1-1"/>
+<wire x1="66.04" y1="16.51" x2="88.59" y2="12.36" width="0" layer="19" extent="1-1"/>
+<wire x1="63.5" y1="7.62" x2="66.04" y2="16.51" width="0" layer="19" extent="1-1"/>
+<wire x1="66.04" y1="5.08" x2="63.5" y2="7.62" width="0" layer="19" extent="1-1"/>
+<wire x1="57.15" y1="11.43" x2="63.5" y2="7.62" width="0" layer="19" extent="1-1"/>
+<wire x1="27.94" y1="16.51" x2="57.15" y2="11.43" width="0" layer="19" extent="1-1"/>
 <wire x1="10.16" y1="12.7" x2="27.94" y2="16.51" width="0" layer="19" extent="1-1"/>
-<wire x1="88.59" y1="28.87" x2="10.16" y2="12.7" width="0" layer="19" extent="1-1"/>
-<wire x1="88.59" y1="12.36" x2="88.59" y2="28.87" width="0" layer="19" extent="1-1"/>
-<wire x1="57.15" y1="11.43" x2="88.59" y2="12.36" width="0" layer="19" extent="1-1"/>
-<wire x1="63.5" y1="7.62" x2="57.15" y2="11.43" width="0" layer="19" extent="1-1"/>
-<wire x1="50.8" y1="2.54" x2="63.5" y2="7.62" width="0" layer="19" extent="1-1"/>
-<wire x1="66.04" y1="5.08" x2="50.8" y2="2.54" width="0" layer="19" extent="1-1"/>
-<wire x1="12.7" y1="36.83" x2="66.04" y2="16.51" width="0" layer="19" extent="1-1"/>
+<wire x1="5.08" y1="24.13" x2="10.16" y2="12.7" width="0" layer="19" extent="1-1"/>
+<wire x1="12.7" y1="36.83" x2="5.08" y2="24.13" width="0" layer="19" extent="1-1"/>
 </signal>
 <signal name="N$9">
@@
 <contactref element="C4" pad="2"/>
 <contactref element="IC2" pad="8"/>
-<wire x1="25.4" y1="24.13" x2="66.04" y2="7.62" width="0" layer="19" extent="1-1"/>
+<contactref element="R12" pad="P$2"/>
+<wire x1="50.8" y1="2.54" x2="66.04" y2="7.62" width="0" layer="19" extent="1-1"/>
+<wire x1="25.4" y1="24.13" x2="50.8" y2="2.54" width="0" layer="19" extent="1-1"/>
 </signal>
 <signal name="N$16">
